Commit message: mapper changes from loc to mapping

File: urdf/t265_tracking_cam_mesh.xacro (robot description, xacro)
@@ -3,8 +3,8 @@
 <!-- _____________________________________________________________________ -->
     <!-- camera_pose_frame link -->
-    <link name="camera_pose_frame"/>
+    <link name="T265_pose_frame"/>
     <!-- camera_pose_frame joint -->
-    <joint name="camera_pose_frame_joint" type="fixed">
-        <parent link="camera_pose_frame"/>
+    <joint name="T265_pose_frame_joint" type="fixed">
+        <parent link="T265_pose_frame"/>
         <child link="base_link"/>
         <origin xyz="0 0 0.030" rpy="0 0 0"/>

File: urdf/t265_tracking_cam_normal.xacro (robot description, xacro)
@@ -2,9 +2,9 @@
 <robot xmlns:xacro="http://www.ros.org/wiki/xacro">
 <!-- _____________________________________________________________________ -->
-    <!-- camera_link link -->
-    <link name="camera_link"/>
-    <!-- camera_link_joint joint -->
-    <joint name="camera_link_joint" type="fixed">
-        <parent link="camera_link"/>
+    <!-- camera_pose_frame link -->
+    <link name="T265_pose_frame"/>
+    <!-- camera_pose_frame joint -->
+    <joint name="T265_pose_frame_joint" type="fixed">
+        <parent link="T265_pose_frame"/>
         <child link="base_link"/>
         <origin xyz="0 0 0.030" rpy="0 0 0"/>
