Commit message: added sim mode

File: urdf/lidar_normal.xacro (robot description, xacro)
@@ -33,7 +33,7 @@
     <!-- LASER FRAME JOINT -->
     <joint name="laser_joint" type="fixed">
-        <parent link="chassis"/>
+        <parent link="base_link"/>
         <child link="laser_frame"/>
-        <origin xyz="0.155 0.0 0.105" rpy="0 0 ${pi}"/>
+        <origin xyz="0.14 0.0 0.105" rpy="0 0 ${pi}"/>
     </joint>
     <!-- LASER FRAME GAZEBO  -->
@@ -54,5 +54,5 @@
                 <range>
                     <min>0.1</min>
-                    <max>5</max>
+                    <max>6</max>
                 </range>
             </ray>

File: urdf/main.urdf.xacro (robot description, xacro)
@@ -1,19 +1,32 @@
 <?xml version="1.0"?>
 <robot xmlns:xacro="http://www.ros.org/wiki/xacro" name="Slambot">
+    <xacro:arg name="sim_mode" default="false"/>          <!-- Use sim_mode when not using real slambot -->
+    <xacro:if value="$(arg sim_mode)">
+        <xacro:include filename="ros2_control_gazebo.xacro" />
+        <xacro:include filename="slambot_normal_version.xacro"/>
+        <xacro:include filename="lidar_normal.xacro"/>
+        <xacro:include filename="t265_tracking_cam_normal.xacro"/>
+    </xacro:if>
+    <xacro:unless value="$(arg sim_mode)">
+        <xacro:include filename="ros2_control_slambot.xacro" />
+        <xacro:include filename="slambot_mesh_version.xacro"/>
+        <xacro:include filename="lidar_mesh.xacro"/>
+        <xacro:include filename="t265_tracking_cam_mesh.xacro"/>
+    </xacro:unless>
 <!-- ___________________________________________Use any one at a time_____________________________________________________________ -->
 <!-- When using gazebo_diff_drive control set "use_ros2_control" to false, and "sim_mode" to true  -->
 <!-- When using ros2_control set "use_ros2_control" to true, and "sim_mode" to true/false based on modes - Real_Robot or Sim_Robot -->
     <!-- <xacro:include filename="ros2_control_gazebo.xacro" /> -->
-    <xacro:include filename="ros2_control_slambot.xacro" />
+    <!-- <xacro:include filename="ros2_control_slambot.xacro" /> -->
 <!-- make sure to comment out the controllers from gazebo_launch of ros2_control when using gazebo_control-->
     <!-- <xacro:include filename="gazebo_control.xacro" />         -->
 <!-- _____________________Use any one model_____________________ -->
 <!--      Normal Version is more compatible with Gazebo Sim      -->
-    <xacro:include filename="slambot_mesh_version.xacro"/>
+    <!-- <xacro:include filename="slambot_mesh_version.xacro"/>
     <xacro:include filename="lidar_mesh.xacro"/>
-    <xacro:include filename="t265_tracking_cam_mesh.xacro"/>
-    <!-- <xacro:include filename="slambot_normal_version.xacro"/> -->
-    <!-- <xacro:include filename="lidar_normal.xacro"/> -->
-    <!-- <xacro:include filename="t265_tracking_cam_normal.xacro"/> -->
+    <xacro:include filename="t265_tracking_cam_mesh.xacro"/> -->
+    <!-- <xacro:include filename="slambot_normal_version.xacro"/>
+    <xacro:include filename="lidar_normal.xacro"/>
+    <xacro:include filename="t265_tracking_cam_normal.xacro"/> -->
 <!-- ____________________________________________________________ -->
     <xacro:include filename="gazebo_config.xacro"/>

File: urdf/ros2_control_gazebo.xacro (robot description, xacro)
@@ -24,6 +24,5 @@
     <gazebo>
         <plugin name="gazebo_ros2_control" filename="libgazebo_ros2_control.so">
-            <parameters>$(find slambot)/config/my_controllers.yaml</parameters>
-            <parameters>$(find slambot)/config/gazebo_ros2_control_w_sim.yaml</parameters>
+            <parameters>$(find slambot)/config/my_controllers_sim.yaml</parameters>
         </plugin>
     </gazebo>

File: urdf/t265_tracking_cam_normal.xacro (robot description, xacro)
@@ -1,17 +1,6 @@
 <?xml version="1.0"?>
 <robot xmlns:xacro="http://www.ros.org/wiki/xacro">
-<!-- _____________________________________________________________________ -->
-    <!-- camera_pose_frame link -->
-    <link name="T265_pose_frame"/>
-    <!-- camera_pose_frame joint -->
-    <joint name="T265_pose_frame_joint" type="fixed">
-        <parent link="T265_pose_frame"/>
-        <child link="base_link"/>
-        <origin xyz="0 0 0.030" rpy="0 0 0"/>
-    </joint>
-<!-- _____________________________________________________________________ -->
-<!-- Custom (just for visual) -->
 <!-- TRACKING CAMERA LINK -->
-<!-- <link name="t265_cam">
+<link name="T265_pose_frame">
     <visual name="">
         <geometry>
@@ -30,10 +19,10 @@
         <origin xyz="0 0 0" rpy="0 0 ${pi/2}"/>
     </xacro:inertial_box>
-</link> -->
+</link>
 <!-- TRACKING CAMERA JOINT -->
-<!-- <joint name="t265_cam_joint" type="fixed">
-    <parent link="chassis"/>
-    <child link="t265_cam"/>
-    <origin xyz="0.19 0 0.0725" rpy="0 0 0"/>
-</joint> -->
+<joint name="T265_pose_frame_joint" type="fixed">
+    <parent link="base_link"/>
+    <child link="T265_pose_frame"/>
+    <origin xyz="0.17 0 0.0725" rpy="0 0 0"/>
+</joint>
 </robot>
